File: Boost.kicad_sch (KiCad schematic)
At the start: 16 parts, among them J1 Conn_01x03, J2 Conn_01x02, Q1 IRF740, U1 MAX1771ESA

Commit message: Added version v0.1-D
- Moved stuff much closer
- Increased the width of the traces
Connections:
- net GND: now also J1.2 (Pin_2), J2.1 (Pin_1); no longer J1.1 (Pin_1), J2.2 (Pin_2)
- net VCC: now also J1.1 (Pin_1); no longer J1.2 (Pin_2)
- net VCC_OUT: now also J2.2 (Pin_2); no longer J2.1 (Pin_1)
- net I_OUT: now reaches D1.2 (A), L1.2, Q1.2 (D)

Commit message: Working on revision 0.1-E
Connections:
- net toggle: now reaches Q1.1 (G), U1.1 (EXT)
Changed lines of the file:
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@@
+		)
+	)
+	(global_label "toggle"
+		(shape input)
+		(at 160.02 92.71 180)
+		(fields_autoplaced yes)
+		(effects
+			(font
+				(size 1.27 1.27)
+			)
+			(justify right)
+		)
+		(property "Intersheetrefs" "${INTERSHEET_REFS}"
+			(at 151.7625 92.71 0)
+			(effects
+				(font
+					(size 1.27 1.27)
+				)
+				(justify right)
+				(hide yes)
+			)
 		)
 	)
